File: PCB/brick-v1.1.kicad_sch (KiCad schematic)
At the start: 53 parts, among them SW1 SW_Push, SW10 SW_Push, SW11 SW_Push, SW12 SW_Push, SW13 SW_Push, SW14 SW_Push, SW15 SW_Push, SW16 SW_Push, SW2 SW_Push, SW3 SW_Push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

Commit message: Redesigned the PCB, and reenamed to macroPAD. Design now features a 2x6 layout and 1 rotary encoder
Connections:
- net at D25.1 (K), D26.1 (K), D27.1 (K)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: no longer U1.9 (GPIO2/SCK)
- net at D17.1 (K), D18.1 (K), D19.1 (K)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: no longer U1.11 (GPIO3/MOSI)
- net at D29.1 (K), D30.1 (K), D31.1 (K)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: no longer U1.8 (GPIO1/RX)
- net at D21.1 (K), D22.1 (K), D23.1 (K)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: no longer U1.10 (GPIO4/MISO)
Changed lines of the file:
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@@
-	(wire
-		(pts
-			(xy 316.23 210.82) (xy 417.83 210.82)
-		)
-		(stroke
-			(width 0)
-			(type default)
-		)
-	)
 	(wire
 		(pts
@@
 	(wire
 		(pts
-			(xy 318.77 292.1) (xy 318.77 213.36)
-		)
-		(stroke
-			(width 0)
-			(type default)
-		)
-	)
-	(wire
-		(pts
 			(xy 520.7 347.98) (xy 520.7 336.55)
 		)
@@
 	(wire
 		(pts
-			(xy 422.91 190.5) (xy 410.21 190.5)
-		)
-		(stroke
-			(width 0)
-			(type default)
-		)
-	)
-	(wire
-		(pts
 			(xy 463.55 317.5) (xy 463.55 323.85)
 		)
@@
 	(wire
 		(pts
-			(xy 312.42 208.28) (xy 415.29 208.28)
-		)
-		(stroke
-			(width 0)
-			(type default)
-		)
-	)
-	(wire
-		(pts
-			(xy 415.29 208.28) (xy 415.29 201.93)
-		)
-		(stroke
-			(width 0)
-			(type default)
-		)
-	)
-	(wire
-		(pts
-			(xy 422.91 217.17) (xy 422.91 190.5)
-		)
-		(stroke
-			(width 0)
-			(type default)
-		)
-	)
-	(wire
-		(pts
 			(xy 431.8 323.85) (xy 463.55 323.85)
 		)
@@
 	(wire
 		(pts
-			(xy 417.83 198.12) (xy 410.21 198.12)
-		)
-		(stroke
-			(width 0)
-			(type default)
-		)
-	)
-	(wire
-		(pts
-			(xy 312.42 304.8) (xy 312.42 208.28)
-		)
-		(stroke
-			(width 0)
-			(type default)
-		)
-	)
-	(wire
-		(pts
 			(xy 214.63 271.78) (xy 214.63 254)
 		)
@@
 	(wire
 		(pts
-			(xy 312.42 304.8) (xy 345.44 304.8)
+			(xy 322.58 304.8) (xy 345.44 304.8)
 		)
 		(stroke
@@
 	(wire
 		(pts
-			(xy 318.77 213.36) (xy 420.37 213.36)
-		)
-		(stroke
-			(width 0)
-			(type default)
-		)
-	)
-	(wire
-		(pts
 			(xy 398.78 347.98) (xy 520.7 347.98)
 		)
@@
 	(wire
 		(pts
-			(xy 322.58 217.17) (xy 422.91 217.17)
-		)
-		(stroke
-			(width 0)
-			(type default)
-		)
-	)
-	(wire
-		(pts
 			(xy 229.87 254) (xy 229.87 237.49)
 		)
@@
 	(wire
 		(pts
-			(xy 322.58 285.75) (xy 322.58 217.17)
-		)
-		(stroke
-			(width 0)
-			(type default)
-		)
-	)
-	(wire
-		(pts
 			(xy 193.04 130.81) (xy 193.04 149.86)
 		)
@@
 	(wire
 		(pts
-			(xy 417.83 210.82) (xy 417.83 198.12)
-		)
-		(stroke
-			(width 0)
-			(type default)
-		)
-	)
-	(wire
-		(pts
 			(xy 242.57 130.81) (xy 243.84 130.81)
 		)
@@
 	(wire
 		(pts
-			(xy 420.37 213.36) (xy 420.37 194.31)
-		)
-		(stroke
-			(width 0)
-			(type default)
-		)
-	)
-	(wire
-		(pts
 			(xy 283.21 237.49) (xy 283.21 220.98)
 		)
@@
 	(wire
 		(pts
-			(xy 420.37 194.31) (xy 410.21 194.31)
-		)
-		(stroke
-			(width 0)
-			(type default)
-		)
-	)
-	(wire
-		(pts
 			(xy 248.92 274.32) (xy 241.3 274.32)
 		)
@@
 	(wire
 		(pts
-			(xy 415.29 201.93) (xy 410.21 201.93)
-		)
-		(stroke
-			(width 0)
-			(type default)
-		)
-	)
-	(wire
-		(pts
 			(xy 322.58 285.75) (xy 417.83 285.75)
 		)
@@
 		)
 	)
-	(wire
-		(pts
-			(xy 316.23 298.45) (xy 316.23 210.82)
-		)
-		(stroke
-			(width 0)
-			(type default)
-		)
-	)
