File: PCB/vali-macroPAD.kicad_sch (KiCad schematic)
At the start: 26 parts, among them SW1 SW_Push, SW10 RotaryEncoder_Switch, SW11 SW_Push, SW12 SW_Push, SW2 SW_Push, SW3 SW_Push, SW4 SW_Push, SW5 SW_Push, SW6 SW_Push, SW7 SW_Push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

Commit message: Created a better case design.
Parts:
- U1: footprint Seeed Studio XIAO Series Library:XIAO-RP2040-DIP -> Hackpad Care Package:XIAO-Generic-Hybrid-14P-2.54-21X17.8MM
Changed lines of the file:
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@@
 	(wire
 		(pts
-			(xy 127 81.28) (xy 132.08 81.28)
+			(xy 83.82 59.69) (xy 83.82 85.09)
 		)
 		(stroke
@@
 	(wire
 		(pts
-			(xy 83.82 59.69) (xy 83.82 85.09)
+			(xy 77.47 16.51) (xy 96.52 16.51)
 		)
 		(stroke
@@
 	(wire
 		(pts
-			(xy 77.47 16.51) (xy 96.52 16.51)
+			(xy 31.75 41.91) (xy 58.42 41.91)
 		)
 		(stroke
@@
 	(wire
 		(pts
-			(xy 31.75 41.91) (xy 58.42 41.91)
+			(xy 64.77 59.69) (xy 64.77 93.98)
 		)
 		(stroke
@@
 	(wire
 		(pts
-			(xy 127 77.47) (xy 127 81.28)
+			(xy 31.75 16.51) (xy 58.42 16.51)
 		)
 		(stroke
@@
 	(wire
 		(pts
-			(xy 64.77 59.69) (xy 64.77 93.98)
+			(xy 83.82 85.09) (xy 83.82 90.17)
 		)
 		(stroke
@@
 	(wire
 		(pts
-			(xy 31.75 16.51) (xy 58.42 16.51)
+			(xy 58.42 41.91) (xy 77.47 41.91)
 		)
 		(stroke
@@
 	(wire
 		(pts
-			(xy 83.82 85.09) (xy 83.82 90.17)
+			(xy 77.47 59.69) (xy 83.82 59.69)
 		)
 		(stroke
@@
 	(wire
 		(pts
-			(xy 58.42 41.91) (xy 77.47 41.91)
+			(xy 58.42 34.29) (xy 64.77 34.29)
 		)
 		(stroke
@@
 	(wire
 		(pts
-			(xy 77.47 59.69) (xy 83.82 59.69)
+			(xy 77.47 67.31) (xy 96.52 67.31)
 		)
 		(stroke
@@
 	(wire
 		(pts
-			(xy 58.42 34.29) (xy 64.77 34.29)
+			(xy 58.42 16.51) (xy 77.47 16.51)
 		)
 		(stroke
@@
 	(wire
 		(pts
-			(xy 77.47 67.31) (xy 96.52 67.31)
+			(xy 64.77 34.29) (xy 64.77 59.69)
 		)
 		(stroke
@@
 	(wire
 		(pts
-			(xy 128.27 73.66) (xy 128.27 77.47)
+			(xy 58.42 59.69) (xy 64.77 59.69)
 		)
 		(stroke
@@
 	(wire
 		(pts
-			(xy 127 73.66) (xy 128.27 73.66)
+			(xy 102.87 34.29) (xy 102.87 59.69)
 		)
 		(stroke
@@
 	(wire
 		(pts
-			(xy 58.42 16.51) (xy 77.47 16.51)
+			(xy 31.75 59.69) (xy 36.83 59.69)
 		)
 		(stroke
@@
 	(wire
 		(pts
-			(xy 64.77 34.29) (xy 64.77 59.69)
+			(xy 102.87 85.09) (xy 102.87 90.17)
 		)
 		(stroke
@@
 	(wire
 		(pts
-			(xy 58.42 59.69) (xy 64.77 59.69)
+			(xy 36.83 34.29) (xy 36.83 59.69)
 		)
 		(stroke
@@
 		)
 	)
-	(wire
-		(pts
-			(xy 128.27 77.47) (xy 132.08 77.47)
-		)
-		(stroke
-			(width 0)
-			(type default)
-		)
-	)
-	(wire
-		(pts
-			(xy 102.87 34.29) (xy 102.87 59.69)
-		)
-		(stroke
-			(width 0)
-			(type default)
-		)
-	)
-	(wire
-		(pts
-			(xy 31.75 59.69) (xy 36.83 59.69)
-		)
-		(stroke
-			(width 0)
-			(type default)
-		)
-	)
-	(wire
-		(pts
-			(xy 102.87 85.09) (xy 102.87 90.17)
-		)
-		(stroke
-			(width 0)
-			(type default)
-		)
-	)
-	(wire
-		(pts
-			(xy 36.83 34.29) (xy 36.83 59.69)
-		)
-		(stroke
-			(width 0)
-			(type default)
-		)
-	)
 	(global_label "Col3"
 		(shape input)
@@
 	(global_label "OLEDSDA"
 		(shape input)
-		(at 127 73.66 180)
+		(at 132.08 77.47 180)
 		(fields_autoplaced yes)
 		(effects
@@
 		)
 		(property "Intersheetrefs" "${INTERSHEET_REFS}"
-			(at 115.6691 73.66 0)
+			(at 120.7491 77.47 0)
 			(effects
 				(font
@@
 	(global_label "OLEDSCL"
 		(shape input)
-		(at 127 77.47 180)
+		(at 132.08 81.28 180)
 		(fields_autoplaced yes)
 		(effects
@@
 		)
 		(property "Intersheetrefs" "${INTERSHEET_REFS}"
-			(at 115.7296 77.47 0)
+			(at 120.8096 81.28 0)
 			(effects
 				(font
@@
 			)
 		)
-		(property "Footprint" "Seeed Studio XIAO Series Library:XIAO-RP2040-DIP"
+		(property "Footprint" "Hackpad Care Package:XIAO-Generic-Hybrid-14P-2.54-21X17.8MM"
 			(at 150.368 89.408 0)
 			(effects
